Commit message: Added bumper

File: environment/robots/urdf/jackal_robot_issac.urdf (robot description, URDF)
Before this commit: robot jackal, 13 links, 12 joints
Links:
- added link sim_collider, mass 1e-5; collision box size=0.52 0.45 0.1
Joints:
- added joint sim_collider_joint: type fixed, parent base_link, child sim_collider, origin xyz=0 0 0 rpy=0 0 0
