Commit message: resloving clash with force plugin and urdf (LiDar)

File: environment/robots/urdf/jackal_robot.urdf (robot description, URDF)
Before this commit: robot jackal, 15 links, 14 joints
Joints:
- joint os1_sensor_joint: parent base_link -> sim_collider

Commit message: jackal_robot collision sensor height correction

File: environment/robots/urdf/jackal_robot.urdf (robot description, URDF)
Before this commit: robot jackal, 15 links, 14 joints
Links:
- link sim_collider: geometry collision box size=0.52 0.45 0.05
Joints:
- joint os1_sensor_joint: origin xyz=0.18 0.0 0.218 rpy=0 0 0 -> xyz=0.18 0.0 0.118 rpy=0 0 0
- joint sim_collider_joint: origin xyz=0 0 0 rpy=0 0 0 -> xyz=0 0 0.10 rpy=0 0 0
