Commit message: xARM6 ISO 23482-1 Sec 7.2 Implementation

File: environment/robots/urdf/xarm6_gripper.urdf (robot description, URDF)
Before this commit: robot xarm6, 17 links, 16 joints
Links:
- added link sim_collider; collision box size=0.05 0.05 0.115
Joints:
- added joint sim_collider_joint: type fixed, parent link6, child sim_collider, origin xyz=0 -0.07 0.11 rpy=0 0 0
