Commit message: sensor plugin

File: environment/robots/urdf/husky.urdf (robot description, URDF)
Before this commit: robot husky, 15 links, 14 joints
Links:
- added link sim_collider, mass 1e-5; collision box size=1.0 0.8 0.1; visual box size=1.0 0.8 0.1
Joints:
- added joint sim_collider_joint: type fixed, parent base_link, child sim_collider, origin xyz=0 0 0 rpy=0 0 0

Commit message: Hidden bumper

File: environment/robots/urdf/husky.urdf (robot description, URDF)
Before this commit: robot husky, 16 links, 15 joints
Links:
- link sim_collider: geometry collision box size=1.0 0.7 0.2

Commit message: Husky ISO 23482-1 Tests till 11.1

File: environment/robots/urdf/husky.urdf (robot description, URDF)
Before this commit: robot husky, 16 links, 15 joints
Links:
- added link os1_sensor, mass 0.33; collision cylinder length=0.073 radius=0.04; visual mesh filename=package://ouster_description/meshes/os1_64.dae
- link sim_collider: geometry collision box size=1.0 0.7 0.02
Joints:
- added joint os1_sensor_joint: type fixed, parent sim_collider, child os1_sensor, origin xyz=0.2 0.0 0.18 rpy=0 0 0
- joint sim_collider_joint: origin xyz=0 0 0 rpy=0 0 0 -> xyz=0 0 0.1 rpy=0 0 0

Commit message: Removed inertial components for contact sensor

File: environment/robots/urdf/husky.urdf (robot description, URDF)
Before this commit: robot husky, 17 links, 16 joints
Links:
- link sim_collider: mass 1e-5 -> None

File: environment/robots/urdf/jackal_robot.urdf (robot description, URDF)
Before this commit: robot jackal, 15 links, 14 joints
Links:
- link sim_collider: mass 1e-5 -> None

Commit message: Modified Huskys force sensor size

File: environment/robots/urdf/husky.urdf (robot description, URDF)
Before this commit: robot husky, 17 links, 16 joints
Links:
- link sim_collider: geometry collision box size=1.0 0.7 0.01
